File: build/kicad/MILESTONE_1_build/full_instrument/full_instrument.kicad_pcb (KiCad board)
At the start: 4 copper layers, 167 x 89.5 mm, 73 parts, among them Q1 S8050 NPN, Q2 S8550 PNP, Q3 S8050, Q4 S8050, Q5 S8050, U1 CD4066, U2 MCP6022, U3 MCP6022, U4 MCP6022, U5 ADS1015, U6 Xiao ESP32-C6

Commit message: update PCB
Routing:
- net Net-(U1-CTLA): track 237.9 -> 211.7 mm
